File: Hardware/Qwiic_PT100.brd (EAGLE design)
At the start: 38.1 x 38.1 mm, 93 parts, among them IC1 ADS122C04IPWR, J2 QWIIC_RIGHT_ANGLE, J3 PTH, J4 QWIIC_RIGHT_ANGLE

Commit message: Remove New-Parts
Parts:
- IC1: device New_Parts:SOP65P640X120-16N -> SparkFun-IC-Conversion:SOP65P640X120-16N
- R9: device New_Parts:0603 -> SparkFun-Resistors:0603
Changed lines of the file:
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@@
 <?xml version="1.0" encoding="utf-8"?>
 <!DOCTYPE eagle SYSTEM "eagle.dtd">
-<eagle version="9.6.0">
+<eagle version="9.6.2">
 <drawing>
 <settings>
@@
 <layer number="128" name="_bValues" color="7" fill="1" visible="no" active="no"/>
 <layer number="129" name="Mask" color="7" fill="1" visible="no" active="no"/>
+<layer number="130" name="SMDSTROOK" color="7" fill="1" visible="no" active="no"/>
 <layer number="131" name="tAdjust" color="7" fill="1" visible="no" active="no"/>
 <layer number="132" name="bAdjust" color="7" fill="1" visible="no" active="no"/>
+<layer number="133" name="bottom_silk" color="7" fill="1" visible="no" active="no"/>
+<layer number="134" name="silk_top" color="7" fill="1" visible="no" active="no"/>
+<layer number="135" name="silk_bottom" color="7" fill="1" visible="no" active="no"/>
+<layer number="136" name="silktop" color="7" fill="1" visible="no" active="no"/>
+<layer number="137" name="silkbottom" color="7" fill="1" visible="no" active="no"/>
+<layer number="138" name="EEE" color="7" fill="1" visible="no" active="no"/>
+<layer number="139" name="_tKeepout" color="7" fill="1" visible="no" active="no"/>
+<layer number="140" name="mbKeepout" color="7" fill="1" visible="no" active="no"/>
+<layer number="141" name="ASSEMBLY_TOP" color="7" fill="1" visible="no" active="no"/>
+<layer number="142" name="mbRestrict" color="7" fill="1" visible="no" active="no"/>
+<layer number="143" name="PLACE_BOUND_TOP" color="7" fill="1" visible="no" active="no"/>
 <layer number="144" name="Drill_legend" color="7" fill="1" visible="no" active="no"/>
+<layer number="145" name="DrillLegend_01-16" color="7" fill="1" visible="no" active="no"/>
+<layer number="146" name="DrillLegend_01-20" color="7" fill="1" visible="no" active="no"/>
+<layer number="147" name="PIN_NUMBER" color="7" fill="1" visible="no" active="no"/>
+<layer number="148" name="DrillLegend_01-20" color="7" fill="1" visible="no" active="no"/>
+<layer number="149" name="DrillLegend_02-15" color="7" fill="1" visible="no" active="no"/>
 <layer number="150" name="Notes" color="7" fill="1" visible="no" active="no"/>
 <layer number="151" name="HeatSink" color="7" fill="1" visible="no" active="no"/>
@@
 <layer number="154" name="FabDoc2" color="7" fill="1" visible="no" active="no"/>
 <layer number="155" name="FabDoc3" color="7" fill="1" visible="no" active="no"/>
+<layer number="166" name="AntennaArea" color="7" fill="1" visible="no" active="no"/>
+<layer number="168" name="4mmHeightArea" color="7" fill="1" visible="no" active="no"/>
+<layer number="191" name="mNets" color="7" fill="1" visible="no" active="no"/>
+<layer number="192" name="mBusses" color="7" fill="1" visible="no" active="no"/>
+<layer number="193" name="mPins" color="7" fill="1" visible="no" active="no"/>
+<layer number="194" name="mSymbols" color="7" fill="1" visible="no" active="no"/>
+<layer number="195" name="mNames" color="7" fill="1" visible="no" active="no"/>
+<layer number="196" name="mValues" color="7" fill="1" visible="no" active="no"/>
 <layer number="199" name="Contour" color="7" fill="1" visible="no" active="no"/>
 <layer number="200" name="200bmp" color="1" fill="10" visible="no" active="no"/>
@@
 <element name="U$39" library="buzzard_labels (66)" package="PWR0" value="" x="1.397" y="30.988" smashed="yes"/>
 <element name="U$40" library="buzzard_labels (66)" package="PWR0" value="" x="1.524" y="21.209" smashed="yes" rot="MR90"/>
-<element name="IC1" library="New_Parts" package="SOP65P640X120-16N" value="ADS122C04IPWR" x="19.05" y="13.97" smashed="yes" rot="R90">
+<element name="IC1" library="SparkFun-IC-Conversion" package="SOP65P640X120-16N" value="ADS122C04IPWR" x="19.05" y="13.97" smashed="yes" rot="R90">
 <attribute name="HEIGHT" value="1.2mm" x="19.05" y="13.97" size="1.778" layer="27" font="vector" ratio="15" rot="R90" display="off"/>
 <attribute name="MANUFACTURER_NAME" value="Texas Instruments" x="19.05" y="13.97" size="1.778" layer="27" font="vector" ratio="15" rot="R90" display="off"/>
@@
 <attribute name="MOUSER_PART_NUMBER" value="595-ADS122C04IPWR" x="19.05" y="13.97" size="1.778" layer="27" font="vector" ratio="15" rot="R90" display="off"/>
 <attribute name="NAME" x="19.431" y="13.97" size="1.27" layer="25" rot="R180" align="center"/>
-<attribute name="PROD_ID" value="" x="19.05" y="13.97" size="1.778" layer="27" rot="R90" display="off"/>
+<attribute name="PROD_ID" value="IC-15119" x="19.05" y="13.97" size="1.778" layer="27" rot="R90" display="off"/>
 </element>
 <element name="JP1" library="SparkFun-Jumpers" package="SMT-JUMPER_3_1-NC_TRACE_SILK" package3d_urn="urn:adsk.eagle:package:39288/1" value="JUMPER-SMT_3_1-NC_TRACE_SILK" x="18.034" y="7.112" smashed="yes" rot="MR180">
@@
 <attribute name="PROD_ID" value="RES-08701" x="23.749" y="16.51" size="1.778" layer="27" ratio="15" rot="R180" display="off"/>
 </element>
-<element name="R9" library="New_Parts" package="0603" value="1620" x="26.67" y="13.97" smashed="yes" rot="R90">
-<attribute name="MOUSER_PART" value="660-RN731JTTD1621B05" x="26.67" y="13.97" size="1.778" layer="27" rot="R90" display="off"/>
+<element name="R9" library="SparkFun-Resistors" package="0603" value="1620" x="26.67" y="13.97" smashed="yes" rot="R90">
 <attribute name="NAME" x="25.908" y="13.97" size="0.6096" layer="25" font="vector" ratio="20" rot="R90" align="bottom-center"/>
-<attribute name="PROD_ID" value=" " x="26.67" y="13.97" size="1.778" layer="27" ratio="15" rot="R90" display="off"/>
-<attribute name="TEMP_COEFF" value="5PPM" x="26.67" y="13.97" size="1.778" layer="27" rot="R90" display="off"/>
-<attribute name="TOLERANCE" value="0.1%" x="26.67" y="13.97" size="1.778" layer="27" rot="R90" display="off"/>
+<attribute name="PROD_ID" value="RES-15120" x="26.67" y="13.97" size="1.778" layer="27" ratio="15" rot="R90" display="off"/>
 <attribute name="VALUE" value="1620" x="27.432" y="13.97" size="0.6096" layer="27" font="vector" ratio="20" rot="R90" align="top-center"/>
 </element>
